File: gameboy-dmg/gameboy-dmg.kicad_pcb (KiCad board)
At the start: 2 copper layers, 82.5 x 77.5 mm, 83 parts, among them J1 Conn_01x02, J3 Conn_01x08, J5 Raspberry_Pi_2_3, J6 Conn_01x09, J7 USB_B_Micro, J8 Conn_01x02, P1 RK10J_POT, SW1 SW_DIP_x01, U1 MCP23017_SO, U2 TP4056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

Commit message: Little board ready for fab
Parts:
- removed the REF** at (179.9, 84.7)
- removed the REF** at (174.9, 92.7)
- removed the REF** at (153.9, 84.6)
- removed the REF** at (127.5, 83.6)
- removed the REF** at (126.0, 78.2)
- removed the REF** at (202.0, 101.8)
- removed the REF** at (202.0, 79.0)
- removed the REF** at (203.2, 92.7)
- removed the REF** at (127.5, 62.5)
- removed the REF** at (201.5, 62.5)
- removed the REF** at (136.9, 115.0)
- removed the REF** at (161.5, 111.7)
- removed the REF** at (148.6, 104.4)
- removed the REF** at (153.4, 107.0)
- removed the REF** at (190.8, 104.8)
- added REF**: MountingHole_2.5mm, MountingHole:MountingHole_2.5mm, F.Cu at (135.9, 100.6)
- added REF**: MountingHole_2.5mm, MountingHole:MountingHole_2.5mm, F.Cu at (130.9, 108.6)
- added REF**: MountingHole_2.5mm, MountingHole:MountingHole_2.5mm, F.Cu at (109.9, 100.5)
- added REF**: MountingHole_2.5mm, MountingHole:MountingHole_2.5mm, F.Cu at (83.5, 99.5)
- added REF**: MountingHole_2.5mm, MountingHole:MountingHole_2.5mm, F.Cu at (82.0, 94.1)
- added REF**: MountingHole_2.5mm, MountingHole:MountingHole_2.5mm, F.Cu at (158.0, 117.7)
- added REF**: MountingHole_2.5mm, MountingHole:MountingHole_2.5mm, F.Cu at (158.0, 94.9)
- added REF**: MountingHole_2.5mm, MountingHole:MountingHole_2.5mm, F.Cu at (159.2, 108.6)
- added REF**: MountingHole_4.5mm, MountingHole:MountingHole_4.5mm, F.Cu at (83.5, 78.4)
- added REF**: MountingHole_4.5mm, MountingHole:MountingHole_4.5mm, F.Cu at (157.5, 78.4)
- added REF**: MountingHole_4.5mm, MountingHole:MountingHole_4.5mm, F.Cu at (92.9, 130.9)
- added REF**: MountingHole_2.5mm, MountingHole:MountingHole_2.5mm, F.Cu at (117.5, 127.6)
- added REF**: MountingHole_2.5mm, MountingHole:MountingHole_2.5mm, F.Cu at (104.6, 120.3)
- added REF**: MountingHole_2.5mm, MountingHole:MountingHole_2.5mm, F.Cu at (109.4, 122.9)
- added REF**: MountingHole_4.5mm, MountingHole:MountingHole_4.5mm, F.Cu at (146.8, 120.7)
- moved P1 50.1 mm to (96.5, 78.5)
- moved C5 46.8 mm to (118.3, 144.5)
- moved J6 46.8 mm to (103.8, 95.2)
- moved JP1 46.8 mm to (101.8, 85.5)
- moved JP10 46.8 mm to (110.3, 77.2)
- moved JP9 46.8 mm to (100.8, 142.4)
- moved R1 46.8 mm to (87.8, 88.2)
- moved RIGHT1 46.8 mm to (103.3, 110.2)
- moved U3 46.8 mm to (90.3, 150.1)
- moved J7 46.8 mm to (115.3, 147.9)
- moved J8 46.8 mm to (122.8, 147.2)
- moved JP6 46.8 mm to (98.3, 96.8)
- moved JP7 46.8 mm to (98.3, 94.3)
- moved A1 46.8 mm to (152.7, 105.3)
- moved B1 46.8 mm to (138.2, 112.1)
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Routing:
- net +3V3: track 41.6 -> 65.9 mm
- net Net-(C8-Pad2): track 13.9 -> 37.5 mm
- net Net-(C2-Pad1): track 5.01 -> 22.0 mm
- net Net-(C7-Pad1): track 16.1 -> 28.7 mm
- net +5V: track 127.6 -> 132.7 mm, vias 2 -> 3
- net Net-(C10-Pad1): track 128.3 -> 125.3 mm
- net Net-(D1-Pad2): track 8.34 -> 5.85 mm
- net /GPIO_SDA_PI: track 13.6 -> 14.7 mm
- net GND: vias 28 -> 29
Other:
- board size 82.5 x 77.5 mm -> 82.5 x 87.5 mm
- board text added: "Volume"
