File: gameboy-dmg-big/MSP_LCD.sch (KiCad schematic (older format))
At the start: 8 parts, among them Q1 S8050, U7 XC6206PxxxMR

Commit message: Big board gerbers
Parts:
- C12: value C_Small -> 100n
Changed lines of the file:
@@
 P 5550 2950
 F 0 "C12" H 5642 2996 50  0000 L CNN
-F 1 "C_Small" H 5642 2905 50  0000 L CNN
+F 1 "100n" H 5642 2905 50  0000 L CNN
 F 2 "Capacitor_SMD:C_0603_1608Metric" H 5550 2950 50  0001 C CNN
 F 3 "~" H 5550 2950 50  0001 C CNN
